File: chronopy.kicad_pcb (KiCad board)
At the start: 2 copper layers, 43 x 43 mm, 78 parts, among them IC1 MCP73831T-2ACI_MC, IC2 S-1000C32-I4T1U, J1 USB_B_Micro, J2 SM02B-SRSS-TB, J3 Conn_01x04_Shielded, Q1 AO3401A, Q2 AO3401A, SW1 SW_DIP_x01, SW2 SW_DIP_x01, SW3 SW_DIP_x01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

Commit message: Update footprint references in schematic and sync
Signed-off-by: Michael Welling <mwelling@ieee.org>
Parts:
- removed the REF** at (139.0, 78.7)
- C1, C10, C13, C14, C15, C16, C2, C3, C4, C5, C6, C7, C8, C9: footprint Badge-PCB:C_0402 -> ChronoPy-PCB:C_0402
- C11, C12: footprint Badge-PCB:C_0805_2012Metric -> ChronoPy-PCB:C_0805_2012Metric
- D1: footprint Badge-PCB:D_SOD-323 -> ChronoPy-PCB:D_SOD-323
- IC1: footprint Badge-PCB:SON50P300X200X100-9N-D -> ChronoPy-PCB:SON50P300X200X100-9N-D
- IC2: footprint Badge-PCB:SNT-4A -> ChronoPy-PCB:SNT-4A
- J1: footprint Badge-PCB:USB_Micro-B_Molex-105017-0001 -> ChronoPy-PCB:USB_Micro-B_Molex-105017-0001
- J2: footprint Badge-PCB:SM02B-SRSS-TB -> ChronoPy-PCB:SM02B-SRSS-TB
- J3: footprint Badge-PCB:JST_SM04B-SRSS-TB(LF)(SN) -> ChronoPy-PCB:JST_SM04B-SRSS-TB(LF)(SN)
- MIC1: footprint Badge-PCB:SPH0645LM4H-B -> ChronoPy-PCB:SPH0645LM4H-B
- Q1, Q2: footprint Badge-PCB:SOT-23 -> ChronoPy-PCB:SOT-23
- R1, R10, R11, R12, R13, R14, R15, R16, R17, R18, R19, R2, R20, R3, R4, R5, R6, R7, R8, R9: footprint Badge-PCB:R_0402 -> ChronoPy-PCB:R_0402
- SW1, SW2, SW3, SW4: footprint Badge-PCB:SW_SPST_TL3305A -> ChronoPy-PCB:SW_SPST_TL3305A
- TFT1: footprint Badge-PCB:0545482271 -> ChronoPy-PCB:0545482271
- TP1, TP10, TP11, TP12, TP2, TP3, TP4, TP5, TP6, TP7, TP8, TP9: footprint Badge-PCB:Test_Point_Pad_d1.0mm -> ChronoPy-PCB:Test_Point_Pad_d1.0mm
- U1: footprint Badge-PCB:SON127P600X500X80-9N -> ChronoPy-PCB:SON127P600X500X80-9N
- U2: footprint Badge-PCB:SOT-23-5 -> ChronoPy-PCB:SOT-23-5
- U3: footprint Badge-PCB:RIGADO_BMD-340-A-R -> ChronoPy-PCB:RIGADO_BMD-340-A-R
- U5: footprint Badge-PCB:PQFN24P43_350X300X102L35X23N -> ChronoPy-PCB:PQFN24P43_350X300X102L35X23N
- U6: footprint Badge-PCB:PSON80P300X300X100-8N -> ChronoPy-PCB:PSON80P300X300X100-8N
- U7: footprint Badge-PCB:APDS-9960 -> ChronoPy-PCB:APDS-9960
- Y1: footprint Badge-PCB:Crystal_SMD_MicroCrystal_CM9V-T1A-2pin_1.6x1.0mm -> ChronoPy-PCB:Crystal_SMD_MicroCrystal_CM9V-T1A-2pin_1.6x1.0mm
