File: chronopy.sch (KiCad schematic (older format))
At the start: 69 parts, among them IC1 MCP73831T-2ACI_MC, IC2 S-1000C32-I4T1U, J1 USB_B_Micro, J2 SM02B-SRSS-TB, J3 Conn_01x04_Shielded, Q1 AO3401A, Q2 AO3401A, SW1 SW_DIP_x01, SW2 SW_DIP_x01, SW3 SW_DIP_x01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

Commit message: Rename everything to ChronoPY and clean up a bit
Signed-off-by: Michael Welling <mwelling@ieee.org>
Parts:
- C1, C10, C13, C14, C15, C16, C2, C3, C4, C5, C6, C7, C8, C9: symbol badge-PCB:C -> ChronoPy-PCB:C
- C11, C12: symbol badge-PCB:CP1 -> ChronoPy-PCB:CP1
- D1: symbol badge-PCB:D -> ChronoPy-PCB:D
- IC1: symbol badge-PCB:MCP73831T-2ACI_MC_MCP73831T-2ACI_MC -> ChronoPy-PCB:MCP73831T-2ACI_MC_MCP73831T-2ACI_MC
- IC2: symbol badge-PCB:S-1000C32-I4T1U_S-1000C32-I4T1U -> ChronoPy-PCB:S-1000C32-I4T1U_S-1000C32-I4T1U
- J1: symbol badge-PCB:USB_B_Micro -> ChronoPy-PCB:USB_B_Micro
- J2: symbol badge-PCB:SM02B-SRSS-TB_LF__SN__SM02B-SRSS-TB -> ChronoPy-PCB:SM02B-SRSS-TB_LF__SN__SM02B-SRSS-TB
- MIC1: symbol badge-PCB:SPH0645LM4H_SPH0645LM4H-B -> ChronoPy-PCB:SPH0645LM4H_SPH0645LM4H-B
- Q1, Q2: symbol badge-PCB:AO3401A-Transistor_FET -> ChronoPy-PCB:AO3401A-Transistor_FET
- R1, R10, R11, R12, R13, R14, R15, R16, R17, R18, R19, R2, R20, R3, R4, R5, R6, R7, R8, R9: symbol badge-PCB:R_US -> ChronoPy-PCB:R_US
- SW1, SW2, SW3, SW4: symbol badge-PCB:SW_DIP_x01 -> ChronoPy-PCB:SW_DIP_x01
- TFT1: symbol badge-PCB:DISP_TFT_1.54IN_240X240_22P-TFT_1.54IN_240X240PIN -> ChronoPy-PCB:DISP_TFT_1.54IN_240X240_22P-TFT_1.54IN_240X240PIN
- TP1, TP10, TP11, TP12, TP2, TP3, TP4, TP5, TP6, TP7, TP8, TP9: symbol badge-PCB:TestPoint-Connector -> ChronoPy-PCB:TestPoint-Connector
- U1: symbol badge-PCB:W25Q32JVSS-Memory_Flash -> ChronoPy-PCB:W25Q32JVSS-Memory_Flash
- U2: symbol badge-PCB:LP2985-3.3 -> ChronoPy-PCB:LP2985-3.3
- U3: symbol badge-PCB:BMD-340-A-R_BMD-340-A-R -> ChronoPy-PCB:BMD-340-A-R_BMD-340-A-R
- U5: symbol badge-PCB:LSM9DS1_LSM9DS1 -> ChronoPy-PCB:LSM9DS1_LSM9DS1
- U6: symbol badge-PCB:BME680_BME680 -> ChronoPy-PCB:BME680_BME680
- U7: symbol badge-PCB:APDS-9960_APDS-9960 -> ChronoPy-PCB:APDS-9960_APDS-9960
- Y1: symbol badge-PCB:Crystal -> ChronoPy-PCB:Crystal

Commit message: Tidy up schematic and add TODO list
Signed-off-by: Michael Welling <mwelling@ieee.org>
Connections:
- wire segments 305 -> 304
Other:
- note added: "1) SWITCH OUT LCD FOR NEW 1.3" CAPTOUCH LCD\n2) SWITCH OUT MICROPHONE FOR PDM ONE\n3) ADD SPEAKER AND/OR VIBRATION MOTOR\n4) CONSIDER SWITCHING TO SIDE SHOOTING BUTTONS\n5) CONSIDER TAG CONNECT FOR SWD"
- note added: "Misc"
- note added: "TODO:"
- moved on the sheet: C1, C10, C11, C12, C13, C14, C15, C16, C2, C9, D1, J3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

Commit message: Update footprint references in schematic and sync
Signed-off-by: Michael Welling <mwelling@ieee.org>
Parts:
- C1, C10, C13, C14, C15, C16, C2, C3, C4, C5, C6, C7, C8, C9: footprint Badge-PCB:C_0402 -> ChronoPy-PCB:C_0402
- C11, C12: footprint Badge-PCB:C_0805_2012Metric -> ChronoPy-PCB:C_0805_2012Metric
- D1: footprint Badge-PCB:D_SOD-323 -> ChronoPy-PCB:D_SOD-323
- IC1: footprint Badge-PCB:SON50P300X200X100-9N-D -> ChronoPy-PCB:SON50P300X200X100-9N-D
- IC2: footprint Badge-PCB:SNT-4A -> ChronoPy-PCB:SNT-4A
- J1: footprint Badge-PCB:USB_Micro-B_Molex-105017-0001 -> ChronoPy-PCB:USB_Micro-B_Molex-105017-0001
- J2: footprint Badge-PCB:SM02B-SRSS-TB -> ChronoPy-PCB:SM02B-SRSS-TB
- J3: footprint Badge-PCB:JST_SM04B-SRSS-TB(LF)(SN) -> ChronoPy-PCB:JST_SM04B-SRSS-TB(LF)(SN)
- MIC1: footprint Badge-PCB:SPH0645LM4H-B -> ChronoPy-PCB:SPH0645LM4H-B
- Q1, Q2: footprint Badge-PCB:SOT-23 -> ChronoPy-PCB:SOT-23
- R1, R10, R11, R12, R13, R14, R15, R16, R17, R18, R19, R2, R20, R3, R4, R5, R6, R7, R8, R9: footprint Badge-PCB:R_0402 -> ChronoPy-PCB:R_0402
- SW1, SW2, SW3, SW4: footprint Badge-PCB:SW_SPST_TL3305A -> ChronoPy-PCB:SW_SPST_TL3305A
- TFT1: footprint Badge-PCB:0545482271 -> ChronoPy-PCB:0545482271
- TP1, TP10, TP11, TP12, TP2, TP3, TP4, TP5, TP6, TP7, TP8, TP9: footprint Badge-PCB:Test_Point_Pad_d1.0mm -> ChronoPy-PCB:Test_Point_Pad_d1.0mm
- U1: footprint Badge-PCB:SON127P600X500X80-9N -> ChronoPy-PCB:SON127P600X500X80-9N
- U2: footprint Badge-PCB:SOT-23-5 -> ChronoPy-PCB:SOT-23-5
- U3: footprint Badge-PCB:RIGADO_BMD-340-A-R -> ChronoPy-PCB:RIGADO_BMD-340-A-R
- U5: footprint Badge-PCB:PQFN24P43_350X300X102L35X23N -> ChronoPy-PCB:PQFN24P43_350X300X102L35X23N
- U6: footprint Badge-PCB:PSON80P300X300X100-8N -> ChronoPy-PCB:PSON80P300X300X100-8N
- U7: footprint Badge-PCB:APDS-9960 -> ChronoPy-PCB:APDS-9960
- Y1: footprint Badge-PCB:Crystal_SMD_MicroCrystal_CM9V-T1A-2pin_1.6x1.0mm -> ChronoPy-PCB:Crystal_SMD_MicroCrystal_CM9V-T1A-2pin_1.6x1.0mm

Commit message: Some updates from the weekend
Signed-off-by: Michael Welling <mwelling@ieee.org>
Parts:
- removed MIC1: SPH0645LM4H-B, ChronoPy-PCB:SPH0645LM4H-B, symbol ChronoPy-PCB:SPH0645LM4H_SPH0645LM4H-B
- removed TFT1: DISP_TFT_1.54IN_240X240_22P, ChronoPy-PCB:0545482271, symbol ChronoPy-PCB:DISP_TFT_1.54IN_240X240_22P-TFT_1.54IN_240X240PIN
- added C17: 0.1uF, ChronoPy-PCB:C_0402, symbol ChronoPy-PCB:C
- added J4: Conn_01x13_MountingPin, ChronoPy-PCB:Hirose_FH26W-13S-0.3SHW_2Rows-13Pins-1MP_P0.60mm, symbol Connector_Generic_MountingPin:Conn_01x13_MountingPin
- added J5: Conn_01x06_MountingPin, ChronoPy-PCB:Hirose_FH19C-6S-0.5SH_1x06-1MP_P0.50mm, symbol Connector_Generic_MountingPin:Conn_01x06_MountingPin
- added J6: Conn_02x05_Odd_Even, Connector_PinHeader_1.27mm:PinHeader_2x05_P1.27mm_Horizontal, symbol Connector_Generic:Conn_02x05_Odd_Even
- added MK1: IM69D120, Sensor_Audio:Infineon_PG-LLGA-5-1, symbol Sensor_Audio:IM69D120
Connections:
- net labels added: GPIO0_15, GPIO0_19, GPIO0_21, GPIO0_24, GPIO0_4, GPIO0_5, GPIO0_6, GPIO0_7, TS_INT, TS_RST
- net labels removed: LCD_TE, MIC_WS
Other:
- note added: "* 1) SWITCH OUT LCD FOR NEW 1.3" CAPTOUCH LCD\n* 2) SWITCH OUT MICROPHONE FOR PDM ONE\n3) ADD SPEAKER AND/OR VIBRATION MOTOR\n4) CONSIDER SWITCHING TO SIDE SHOOTING BUTTONS\n5) CONSIDER TAG CONNECT FOR SWD\n* 6) ADD MORE EXPANSION HEADERS"
- note added: "IIC addr: 0x76"
- note removed: "1) SWITCH OUT LCD FOR NEW 1.3" CAPTOUCH LCD\n2) SWITCH OUT MICROPHONE FOR PDM ONE\n3) ADD SPEAKER AND/OR VIBRATION MOTOR\n4) CONSIDER SWITCHING TO SIDE SHOOTING BUTTONS\n5) CONSIDER TAG CONNECT FOR SWD"
- note removed: "IIC: 0x76"
- note removed: "Mic, Optional, nice to have"
- moved on the sheet: C10, C11, C12, C13, C14, C15, C16, C9, J3, Q2, R10, R11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

Commit message: Added Fuel Gauge IC
Parts:
- added Q?: Q_NMOS_GDS, symbol Device:Q_NMOS_GDS
- added Q?: AO3401A, ChronoPy-PCB:SOT-23, symbol ChronoPy-PCB:AO3401A-Transistor_FET
- added R? (x2): 100k, ChronoPy-PCB:R_0402, symbol ChronoPy-PCB:R_US
- added R?: 22, ChronoPy-PCB:R_0402, symbol ChronoPy-PCB:R_US
- added U?: STC3117IJT, symbol ChronoPy-PCB:STC3117IJT
- IC2: value S-1000C32-I4T1U -> S-1000C32-I4T1U_S-1000C32-I4T1U; footprint ChronoPy-PCB:SNT-4A -> SNT-4A
Connections:
- net labels added: CHG_INHB
- wire segments 304 -> 323
Other:
- moved on the sheet: C3, C5, IC1, J2, R14, R20, R4, R5

Commit message: Clean up schematic changes for fuel gauge
Cleans schematic a bit and start the layout for the fuel gauge.

Signed-off-by: Michael Welling <mwelling@ieee.org>
Parts:
- removed Q?: Q_NMOS_GDS, symbol Device:Q_NMOS_GDS
- removed Q?: AO3401A, ChronoPy-PCB:SOT-23, symbol ChronoPy-PCB:AO3401A-Transistor_FET
- removed R?: 22, ChronoPy-PCB:R_0402, symbol ChronoPy-PCB:R_US
- added C18: 220nF, ChronoPy-PCB:C_0402, symbol ChronoPy-PCB:C
- added C19: 1uF, ChronoPy-PCB:C_0402, symbol ChronoPy-PCB:C
- added R22: 1k, ChronoPy-PCB:R_0402, symbol ChronoPy-PCB:R_US
- MK1: symbol Sensor_Audio:IM69D120 -> chronopy-rescue:IM69D120-Sensor_Audio
- R21: renamed from R?; value 100k -> 1k
- R23: renamed from R?; value 100k -> 10m 1%; footprint ChronoPy-PCB:R_0402 -> Resistor_SMD:R_0603_1608Metric
- U4: renamed from U?; footprint (none) -> ChronoPy-PCB:CSP-9
Connections:
- wire segments 323 -> 325
Other:
- moved on the sheet: C1, C2, C3, C4, C5, C6, C7, C8, D1, IC1, IC2, J1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

Commit message: Adds new fuel gauge and vibration motor
Signed-off-by: Michael Welling <mwelling@ieee.org>
Parts:
- removed U4: STC3117IJT, ChronoPy-PCB:CSP-9, symbol ChronoPy-PCB:STC3117IJT
- added D2: D, ChronoPy-PCB:D_SOD-323, symbol ChronoPy-PCB:D
- added M1: Z43FC1B5640007L, ChronoPy-PCB:Z43FC1B5640007L, symbol Motor:Motor_DC_ALT
- added Q3: AO3401A, ChronoPy-PCB:SOT-23, symbol ChronoPy-PCB:AO3401A-Transistor_FET
- added R24: 100k, ChronoPy-PCB:R_0402, symbol ChronoPy-PCB:R_US
- added U4: STC3115IJT, ChronoPy-PCB:CSP-10, symbol ChronoPy-PCB:STC3115IJT
Connections:
- net +3V0: now also Q3.2 (S), R24.1
- net +BATT: now also U4.B3 (VCC)
- net GND: now also D2.2 (A), M1.2 (-), U4.C3 (RSTIO), U4.D1 (GND)
- net IIC_SCL: now also U4.C1 (SCL)
- net IIC_SDA: now also U4.B1 (SDA)
- net SW_A: now also U3.9 (P0.28); no longer U3.10 (P0.29)
- net at J2.1, R23.2: now also U4.D3 (CG)
- net at R21.1: now also U4.B2 (BATD/CD)
- net at C18.1, R22.1: now also U4.A3 (VIN)
- net CHG_INHB: no longer names the net of IC1.8 (PROG), R4.2
- new net: D2.1 (K), M1.1 (+), Q3.3 (D)
- new net MOTOR_EN: Q3.1 (G), R24.2, U3.10 (P0.29)
Other:
- note added: "* 1) SWITCH OUT LCD FOR NEW 1.3" CAPTOUCH LCD\n* 2) SWITCH OUT MICROPHONE FOR PDM ONE\n* 3) ADD SPEAKER AND/OR VIBRATION MOTOR\n4) CONSIDER SWITCHING TO SIDE SHOOTING BUTTONS\n5) CONSIDER TAG CONNECT FOR SWD\n* 6) ADD MORE EXPANSION HEADERS"
- note added: "Vibration Motor"
- note removed: "* 1) SWITCH OUT LCD FOR NEW 1.3" CAPTOUCH LCD\n* 2) SWITCH OUT MICROPHONE FOR PDM ONE\n3) ADD SPEAKER AND/OR VIBRATION MOTOR\n4) CONSIDER SWITCHING TO SIDE SHOOTING BUTTONS\n5) CONSIDER TAG CONNECT FOR SWD\n* 6) ADD MORE EXPANSION HEADERS"
Changed lines of the file:
@@
 Text GLabel 12900 3600 1    50   Input ~ 0
 SW_B
-Text GLabel 5350 9900 2    50   Input ~ 0
+Text GLabel 5350 10000 2    50   Input ~ 0
 SW_A
 Text GLabel 4050 8900 0    50   Input ~ 0
@@
 Wire Wire Line
 	5350 8300 5250 8300
-Wire Wire Line
-	5250 8400 5350 8400
 Wire Wire Line
 	4150 10300 4000 10300
@@
 TODO:
 Text Notes 1300 14450 0    157  ~ 0
-* 1) SWITCH OUT LCD FOR NEW 1.3" CAPTOUCH LCD\n* 2) SWITCH OUT MICROPHONE FOR PDM ONE\n3) ADD SPEAKER AND/OR VIBRATION MOTOR\n4) CONSIDER SWITCHING TO SIDE SHOOTING BUTTONS\n5) CONSIDER TAG CONNECT FOR SWD\n* 6) ADD MORE EXPANSION HEADERS
+* 1) SWITCH OUT LCD FOR NEW 1.3" CAPTOUCH LCD\n* 2) SWITCH OUT MICROPHONE FOR PDM ONE\n* 3) ADD SPEAKER AND/OR VIBRATION MOTOR\n4) CONSIDER SWITCHING TO SIDE SHOOTING BUTTONS\n5) CONSIDER TAG CONNECT FOR SWD\n* 6) ADD MORE EXPANSION HEADERS
 Connection ~ 6050 1650
 $Comp
@@
 	0    -1   -1   0
 $EndComp
-$Comp
-L ChronoPy-PCB:STC3117IJT U4
-U 1 1 5F71B978
-P 3600 5850
-F 0 "U4" H 3600 6465 50  0000 C CNN
-F 1 "STC3117IJT" H 3600 6374 50  0000 C CNN
-F 2 "ChronoPy-PCB:CSP-9" H 3650 6600 50  0001 C CNN
-F 3 "" H 3650 6600 50  0001 C CNN
-	1    3600 5850
-	1    0    0    -1
-$EndComp
 Connection ~ 3000 3800
 $Comp
@@
 Wire Wire Line
 	4050 6150 4150 6150
-$Comp
-L power:GND #PWR022
-U 1 1 5F8CD3DA
-P 4600 6150
-F 0 "#PWR022" H 4600 5900 50  0001 C CNN
-F 1 "GND" H 4605 5977 50  0000 C CNN
-F 2 "" H 4600 6150 50  0001 C CNN
-F 3 "" H 4600 6150 50  0001 C CNN
-	1    4600 6150
-	0    -1   -1   0
-$EndComp
-Wire Wire Line
-	4600 6150 4450 6150
 Text GLabel 3050 6250 0    50   Input ~ 0
 IIC_SCL
@@
 Wire Wire Line
 	3050 6350 3150 6350
-Wire Wire Line
-	5200 5950 5200 6250
-Text GLabel 3050 5500 0    50   Input ~ 0
-CHG_INHB
-Text GLabel 4350 3550 2    50   Input ~ 0
-CHG_INHB
 Wire Wire Line
 	4200 4000 4800 4000
@@
 	4900 5500 5200 5500
 Wire Wire Line
-	4350 3550 4250 3550
-Wire Wire Line
-	4200 3800 4250 3800
-Wire Wire Line
 	4800 3800 4650 3800
-Wire Wire Line
-	3050 5500 3150 5500
-Wire Wire Line
-	4250 3550 4250 3800
-Connection ~ 4250 3800
-Wire Wire Line
-	4250 3800 4350 3800
+$Comp
+L ChronoPy-PCB:STC3115IJT U4
+U 1 1 5FC3EFC2
+P 3600 5850
+F 0 "U4" H 3600 6470 50  0000 C CNN
+F 1 "STC3115IJT" H 3600 6379 50  0000 C CNN
+F 2 "ChronoPy-PCB:CSP-10" H 3650 6600 50  0001 C CNN
+F 3 "" H 3650 6600 50  0001 C CNN
+	1    3600 5850
+	1    0    0    -1
+$EndComp
+Wire Wire Line
+	5200 5950 5200 6250
+$Comp
+L power:GND #PWR0129
+U 1 1 5FC5D4DB
+P 4650 6150
+F 0 "#PWR0129" H 4650 5900 50  0001 C CNN
+F 1 "GND" V 4650 5950 50  0000 C CNN
+F 2 "" H 4650 6150 50  0001 C CNN
+F 3 "" H 4650 6150 50  0001 C CNN
+	1    4650 6150
+	0    -1   -1   0
+$EndComp
+Wire Wire Line
+	4450 6150 4650 6150
+Wire Wire Line
+	4200 3800 4350 3800
+$Comp
+L power:GND #PWR0130
+U 1 1 5FC79D83
+P 3000 5600
+F 0 "#PWR0130" H 3000 5350 50  0001 C CNN
+F 1 "GND" H 3005 5427 50  0000 C CNN
+F 2 "" H 3000 5600 50  0001 C CNN
+F 3 "" H 3000 5600 50  0001 C CNN
+	1    3000 5600
+	1    0    0    -1
+$EndComp
+Wire Wire Line
+	3150 5500 3000 5500
+Wire Wire Line
+	3000 5500 3000 5600
+$Comp
+L Motor:Motor_DC_ALT M1
+U 1 1 5FCD5516
+P 17450 3950
+F 0 "M1" H 17597 3946 50  0000 L CNN
+F 1 "Z43FC1B5640007L" H 17597 3855 50  0000 L CNN
+F 2 "ChronoPy-PCB:Z43FC1B5640007L" H 17450 3860 50  0001 C CNN
+F 3 "~" H 17450 3860 50  0001 C CNN
+	1    17450 3950
+	1    0    0    -1
+$EndComp
+$Comp
+L ChronoPy-PCB:R_US R24
+U 1 1 5FD2F170
+P 16100 3900
+F 0 "R24" H 15950 3850 50  0000 C CNN
+F 1 "100k" H 15950 3950 50  0000 C CNN
+F 2 "ChronoPy-PCB:R_0402" V 16140 3890 50  0001 C CNN
+F 3 "~" H 16100 3900 50  0001 C CNN
+	1    16100 3900
+	1    0    0    -1
+$EndComp
+Text GLabel 16100 4200 3    50   Input ~ 0
+MOTOR_EN
+$Comp
+L ChronoPy-PCB:AO3401A-Transistor_FET Q3
+U 1 1 5FD2F178
+P 16550 3800
+F 0 "Q3" V 16892 3800 50  0000 C CNN
+F 1 "AO3401A" V 16801 3800 50  0000 C CNN
+F 2 "ChronoPy-PCB:SOT-23" H 16750 3725 50  0001 L CIN
+F 3 "http://www.aosmd.com/pdfs/datasheet/AO3401A.pdf" H 16550 3800 50  0001 L CNN
+	1    16550 3800
+	0    1    -1   0
+$EndComp
+$Comp
+L ChronoPy-PCB:+3V0-power #PWR022
+U 1 1 5FD2F17F
+P 16100 3600
+F 0 "#PWR022" H 16100 3450 50  0001 C CNN
+F 1 "+3V0" H 16115 3773 50  0000 C CNN
+F 2 "" H 16100 3600 50  0001 C CNN
+F 3 "" H 16100 3600 50  0001 C CNN
+	1    16100 3600
+	1    0    0    -1
+$EndComp
+Wire Wire Line
+	16350 3700 16100 3700
+Wire Wire Line
+	16100 3700 16100 3600
+Wire Wire Line
+	16100 3750 16100 3700
+Connection ~ 16100 3700
+Wire Wire Line
+	16100 4200 16100 4100
+Wire Wire Line
+	16100 4100 16550 4100
+Wire Wire Line
+	16550 4100 16550 4000
+Connection ~ 16100 4100
+Wire Wire Line
+	16100 4100 16100 4050
+Wire Wire Line
+	17450 3700 17450 3750
+$Comp
+L power:GND #PWR025
+U 1 1 5FD67D38
+P 17450 4350
+F 0 "#PWR025" H 17450 4100 50  0001 C CNN
+F 1 "GND" V 17455 4222 50  0000 R CNN
+F 2 "" H 17450 4350 50  0001 C CNN
+F 3 "" H 17450 4350 50  0001 C CNN
+	1    17450 4350
+	1    0    0    -1
+$EndComp
+Wire Wire Line
+	17450 4250 17450 4300
+Text GLabel 5350 9900 2    50   Input ~ 0
+MOTOR_EN
+Wire Wire Line
+	17100 3850 17100 3700
+Wire Wire Line
+	17100 3700 17450 3700
+Wire Wire Line
+	17450 4300 17100 4300
+Wire Wire Line
+	17100 4300 17100 4150
+Connection ~ 17450 4300
+Wire Wire Line
+	17450 4300 17450 4350
+Wire Wire Line
+	16750 3700 17100 3700
+Connection ~ 17100 3700
+$Comp
+L ChronoPy-PCB:D D2
+U 1 1 5FF1D702
+P 17100 4000
+F 0 "D2" H 17100 4100 50  0000 C CNN
+F 1 "D" H 17100 4100 50  0001 C CNN
+F 2 "ChronoPy-PCB:D_SOD-323" H 17100 4000 50  0001 C CNN
+F 3 "~" H 17100 4000 50  0001 C CNN
+	1    17100 4000
+	0    1    1    0
+$EndComp
+Wire Notes Line
+	15350 2900 18450 2900
+Wire Notes Line
+	18450 2900 18450 4750
+Wire Notes Line
+	15350 2900 15350 4750
+Wire Notes Line
+	15350 4750 18450 4750
+Text Notes 15550 3200 0    157  ~ 0
+Vibration Motor
 $EndSCHEMATC

Commit message: Switch to side shooter buttons and add Tag connect
Signed-off-by: Michael Welling <mwelling@ieee.org>
Parts:
- removed TP1, TP11, TP2: TestPoint, ChronoPy-PCB:Test_Point_Pad_d1.0mm, symbol ChronoPy-PCB:TestPoint-Connector
- added J7: TC2030-CTX, ChronoPy-PCB:TC2030-IDC-NL, symbol ChronoPy-PCB:TC2030-CTX
- SW1, SW2, SW3, SW4: footprint ChronoPy-PCB:SW_SPST_TL3305A -> ChronoPy-PCB:SW_TL3340AF160QG
Connections:
- net +3V0: now also J7.1 (VCC)
- net GND: now also SW1.1, SW2.1, SW3.1, SW4.1, J7.5 (GND); no longer SW1.2, SW2.2, SW3.2, SW4.2
- net SWCLK: now also J7.4 (TCK)
- net SWDIO: now also J7.2 (TMS)
- net SW_A: now also SW1.2; no longer SW1.1
- net SW_B: now also SW2.2; no longer SW2.1
- net SW_C: now also SW3.2; no longer SW3.1
- net SW_D: now also SW4.2; no longer SW4.1
- net ~RESET: now also J7.3 (~RESET)
Other:
- note added: "TAG Connect"
- note removed: "* 1) SWITCH OUT LCD FOR NEW 1.3" CAPTOUCH LCD\n* 2) SWITCH OUT MICROPHONE FOR PDM ONE\n* 3) ADD SPEAKER AND/OR VIBRATION MOTOR\n4) CONSIDER SWITCHING TO SIDE SHOOTING BUTTONS\n5) CONSIDER TAG CONNECT FOR SWD\n* 6) ADD MORE EXPANSION HEADERS"
- note removed: "TODO:"
- moved on the sheet: TP10, TP12, TP3, TP4, TP5, TP6, TP7, TP8, TP9
